Commit message: probando2

File: pybullet/urdf/practica0.urdf (robot description, URDF)
Before this commit: robot trifasiko, 3 links, 2 joints
Joints:
- joint base_to_long: type revolute -> fixed

Commit message: acabado?

File: pybullet/urdf/practica0.urdf (robot description, URDF)
Before this commit: robot trifasiko, 3 links, 2 joints
Joints:
- joint long_to_short: limit lower=-1.0 upper=1.0 effort=1000.0 velocity=0.5 -> lower=4.0 upper=-4.0 effort=1000.0 velocity=0.5

Commit message: b

File: pybullet/urdf/practica0.urdf (robot description, URDF)
Before this commit: robot trifasiko, 3 links, 2 joints
Joints:
- joint base_to_long: type fixed -> revolute

Commit message: FIN PRAC0

File: pybullet/urdf/practica0.urdf (robot description, URDF)
Before this commit: robot trifasiko, 3 links, 2 joints
Links:
- link short_arm: mass 200.0 -> 2.0
