Commit message: escenario final

File: pybullet/urdf/barrita.urdf (robot description, URDF)
Before this commit: robot barrita, 2 links, 1 joints
Links:
- link barra: mass 2.0 -> 5.0; geometry collision box size=0.1 2.0 0.1; visual box size=0.1 2.0 0.1
- link cilindro: mass 20000.0 -> 200000.0; geometry collision cylinder length=1.0 radius=0.2; visual cylinder length=1.0 radius=0.2
Joints:
- joint not_to_pass: origin xyz=0.0 0.0 0.0 rpy=0.0 0.0 0.0 -> xyz=0.0 0.0 0.0 rpy=0 0.0 -3.15/2

File: pybullet/urdf/final.urdf (robot description, URDF)
Before this commit: robot final, 1 links, 0 joints
Links:
- link meta: geometry collision box size=1.0 3.5 0.10; visual box size=1.0 3.5 0.10

Commit message: Añadido Fase 3 y 4

File: pybullet/urdf/barrita.urdf (robot description, URDF)
Before this commit: robot barrita, 2 links, 1 joints
Links:
- link cilindro: mass 200000.0 -> 300.0
Joints:
- joint not_to_pass: origin xyz=0.0 0.0 0.0 rpy=0 0.0 -3.15/2 -> xyz=0.0 0.0 0.0 rpy=0 0.0 -3.15

File: pybullet/urdf/final.urdf (robot description, URDF)
Before this commit: robot final, 1 links, 0 joints
Links:
- link meta: geometry collision box size=1.0 3.5 0.01; visual box size=1.0 3.5 0.01

Commit message: cambio friccion

File: pybullet/urdf/barrita.urdf (robot description, URDF)
Before this commit: robot barrita, 2 links, 1 joints
Joints:
- joint not_to_pass: origin xyz=0.0 0.0 0.0 rpy=0 0.0 -3.15 -> xyz=0.0 0.0 0.0 rpy=0 0.0 0

Commit message: BUG BARRITA

File: pybullet/urdf/barrita.urdf (robot description, URDF)
Before this commit: robot barrita, 2 links, 1 joints
Links:
- link cilindro: geometry collision cylinder length=1.0 radius=0.2; visual cylinder length=1.1 radius=0.2
