Commit message: rover.joints

File: urdf/robot_nuevo.urdf (robot description, URDF)
Before this commit: robot robot_nuevo, 12 links, 11 joints
Links:
- removed link Untitled.007
- removed link Untitled.008
- removed link Untitled.009
- removed link pinzaL
- removed link pinzaR
- removed link sphere
- added link Untitled, mass 0.001; collision box size=0.5 0.3 2.41; visual box size=0.5 0.3 2.41
- added link Untitled.001, mass 0.001; collision box size=0.45 0.61 0.02; visual box size=0.45 0.61 0.02
- added link Untitled.002, mass 0.001; collision box size=0.9 0.61 0.11; visual box size=0.9 0.61 0.11
- added link Untitled.003, mass 0.001; collision box size=0.45 0.61 0.02; visual box size=0.45 0.61 0.02
- added link Untitled.004, mass 0.001; collision box size=0.5 0.3 1.87; visual box size=0.5 0.3 1.9
- added link Untitled.005, mass 0.001; collision box size=0.5 0.3 3.25; visual box size=0.5 0.3 3.25
- link Untitled.006: geometry collision sphere radius=0.5; visual mesh filename=../meshes/dae/Sphere.dae scale=0.5 0.5 0.5
- link coche: mass 0.001 -> 10000.0; geometry collision mesh filename=../meshes/dae/Cube.016.dae scale=1.0 1.0 1.0; visual mesh filename=../meshes/dae/Cube.dae scale=1.0 1.715 0.78246
- link rueda1: geometry collision mesh filename=../meshes/dae/Torus.001.dae scale=1.0 1.0 1.0; visual mesh filename=../meshes/dae/Torus.007.dae scale=0.4 0.4 1.0
- link rueda2: geometry collision mesh filename=../meshes/dae/Torus.000.dae scale=1.0 1.0 1.0; visual mesh filename=../meshes/dae/Torus.008.dae scale=0.4 0.4 1.0
- link rueda3: geometry collision mesh filename=../meshes/dae/Torus.004.dae scale=1.0 1.0 1.0; visual mesh filename=../meshes/dae/Torus.003.dae scale=0.4 0.4 1.0
- link rueda4: geometry collision mesh filename=../meshes/dae/Torus.002.dae scale=1.0 1.0 1.0; visual mesh filename=../meshes/dae/Torus.006.dae scale=0.4 0.4 1.0
Joints:
- removed joint Untitled.007
- removed joint Untitled.008
- removed joint Untitled.009
- removed joint pinzaL
- removed joint pinzaR
- removed joint sphere
- added joint Untitled: type prismatic, parent coche, child Untitled, origin xyz=0 -1.3 1.50313 rpy=0 0 0, axis 0 0 1.0, limit lower=0 upper=0 effort=0 velocity=0
- added joint Untitled.001: type floating, parent Untitled.005, child Untitled.001, origin xyz=-3.07181 -2.04296 -0.35164 rpy=-0.02845 0 -1.5708
- added joint Untitled.002: type floating, parent Untitled.005, child Untitled.002, origin xyz=-3.05929 -1.78296 0.08819 rpy=-1.5708 -1.54235 0
- added joint Untitled.003: type floating, parent Untitled.005, child Untitled.003, origin xyz=-3.04678 -2.04296 0.52801 rpy=-0.02845 0 -1.5708
- added joint Untitled.004: type floating, parent Untitled.005, child Untitled.004, origin xyz=-3.04707 -1.00568 0.08784 rpy=-1.5708 -1.54235 0
- added joint Untitled.005: type revolute, parent Untitled.006, child Untitled.005, origin xyz=0.03695 -0.02274 0.42047 rpy=1.5708 0 2.18414, axis 0 0 1.0, limit lower=1.5708 upper=0 effort=0 velocity=0
- joint Untitled.006: limit lower=0 upper=0 effort=0 velocity=0 -> effort=0 velocity=0; origin xyz=0 -1.3 1.59275 rpy=0 0 0 -> xyz=-0.01713 0.0009 0.84188 rpy=0 0 0; parent coche -> Untitled; type prismatic -> continuous
