Commit message: modificado diseño

File: urdf/probando.urdf (robot description, URDF)
Before this commit: robot robot_nuevo, 12 links, 11 joints
Links:
- removed link Untitled
- removed link Untitled.001
- removed link Untitled.003
- removed link Untitled.004
- removed link Untitled.005
- removed link Untitled.006
- added link Barra_principal, mass 30.0; collision box size=0.5 0.3 2.41; visual box size=0.5 0.3 2.41
- added link Pinza_L, mass 15.51; collision box size=0.45 0.61 0.02; visual box size=0.45 0.61 0.02
- added link Pinza_R, mass 15.51; collision box size=0.45 0.61 0.02; visual box size=0.45 0.61 0.02
- added link barra_gira, mass 30.0; collision box size=0.5 0.3 2.17; visual box size=0.5 0.30001 2.17
- added link barra_pinza, mass 20.0; collision box size=0.5 0.3 2.7; visual box size=0.5 0.3 2.74
- added link esfera, mass 30.0; collision sphere radius=0.5; visual mesh filename=../meshes/dae/Sphere.dae scale=0.5 0.5 0.5
- link rueda1: mass 0.001 -> 10.0
- link rueda2: mass 0.001 -> 10.0
- link rueda3: mass 0.001 -> 10.0
- link rueda4: mass 0.001 -> 10.0
Joints:
- removed joint Untitled
- removed joint Untitled.001
- removed joint Untitled.003
- removed joint Untitled.004
- removed joint Untitled.005
- removed joint Untitled.006
- added joint Barra_principal: type prismatic, parent coche, child Barra_principal, origin xyz=0 -1.3 1.50313 rpy=0 0 0, axis 0 0 1.0, limit lower=-0.82 upper=0.5 effort=0 velocity=0
- added joint Pinza_L: type prismatic, parent Untitled.002, child Pinza_L, origin xyz=-0.39871 0.01611 -0.26543 rpy=3.14159 1.5708 0, axis 0 0 1.0, limit lower=1.92 upper=0.03 effort=0 velocity=0
- added joint Pinza_R: type prismatic, parent Untitled.002, child Pinza_R, origin xyz=0.44 0 -0.26 rpy=0 1.5708 0, axis 0 0 1.0, limit lower=-0.15 upper=0 effort=0 velocity=0
- added joint barra_gira: type fixed, parent esfera, child barra_gira, origin xyz=0.03695 -0.02274 0.17047 rpy=1.5708 0 2.18414
- added joint barra_pinza: type prismatic, parent barra_gira, child barra_pinza, origin xyz=-1.83756 -0.82282 0.05342 rpy=-1.5708 -1.54235 0, axis 0 0 1.0, limit lower=-1.17 upper=0.9 effort=0 velocity=0
- added joint esfera: type continuous, parent Barra_principal, child esfera, origin xyz=-0.01713 0.0009 0.84188 rpy=0 0 0, axis 0 0 1.0, limit effort=0 velocity=0
- joint Untitled.002: origin xyz=-3.05929 -1.78296 0.08819 rpy=-1.5708 -1.54235 0 -> xyz=0 -0.01222 -0.7498 rpy=0 0 0; parent Untitled.005 -> barra_pinza
